File: PCB_Sensor.kicad_pcb (KiCad board)
At the start: 2 copper layers, 88.9 x 88.9 mm, 38 parts, among them J1 DHT22, J10 PRGM, J11 UWB, J12 LCDDATA, J13 LCDTOUCH, J14 ESP01A, J15 ESP01B, J2 VOLTSENSOR, J4 COM, J5 ALERT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

Commit message: generate gerber file
Other:
- board text added: "ASTAR TECH"
- board text added: "by Greatreyhan"

Commit message: update
Parts:
- added J16: DRV_B, TerminalBlock:TerminalBlock_bornier-2_P5.08mm, F.Cu at (63.5, 142.2)
- added J17: DRV_C, TerminalBlock:TerminalBlock_bornier-2_P5.08mm, F.Cu at (170.2, 43.2)
- added J18: DRV_D, TerminalBlock:TerminalBlock_bornier-2_P5.08mm, F.Cu at (170.2, 142.2)
- added J19: MTR_A, TerminalBlock:TerminalBlock_bornier-2_P5.08mm, F.Cu at (63.5, 43.2)
- added J20: MTR_B, TerminalBlock:TerminalBlock_bornier-2_P5.08mm, F.Cu at (63.5, 85.5)
- added J21: MTR_C, TerminalBlock:TerminalBlock_bornier-2_P5.08mm, F.Cu at (63.5, 96.5)
- added J22: MTR_D, TerminalBlock:TerminalBlock_bornier-2_P5.08mm, F.Cu at (63.5, 107.5)
- added J23: DRV_ENCA, Connector_PinHeader_2.54mm:PinHeader_1x04_P2.54mm_Vertical, F.Cu at (162.6, 35.6)
- added J24: DRV_ENCB, Connector_PinHeader_2.54mm:PinHeader_1x04_P2.54mm_Vertical, F.Cu at (154.9, 144.8)
- added J25: DRV_ENCC, Connector_PinHeader_2.54mm:PinHeader_1x04_P2.54mm_Vertical, F.Cu at (78.7, 35.6)
- added J26: DRV_ENCD, Connector_PinHeader_2.54mm:PinHeader_1x04_P2.54mm_Vertical, F.Cu at (71.1, 144.8)
- added J27: ENCA, Connector_PinHeader_2.54mm:PinHeader_1x04_P2.54mm_Vertical, F.Cu at (170.2, 63.5)
- added J28: ENCC, Connector_PinHeader_2.54mm:PinHeader_1x04_P2.54mm_Vertical, F.Cu at (170.2, 76.2)
- added J29: ENCB, Connector_PinHeader_2.54mm:PinHeader_1x04_P2.54mm_Vertical, F.Cu at (170.2, 101.6)
- added J3: DRV_A, TerminalBlock:TerminalBlock_bornier-2_P5.08mm, F.Cu at (63.5, 74.5)
- added J30: ENCD, Connector_PinHeader_2.54mm:PinHeader_1x04_P2.54mm_Vertical, F.Cu at (170.2, 88.9)
- moved BZ1 25.4 mm to (135.9, 109.2)
- moved J10 25.4 mm to (157.5, 121.9)
- moved J12 25.4 mm to (157.5, 94.0)
- moved J14 25.4 mm to (137.2, 71.1)
- moved J4 25.4 mm to (157.5, 66.0)
- moved J7 25.4 mm to (111.8, 76.2)
- moved J9 25.4 mm to (94.0, 116.8)
- moved R1 25.4 mm to (130.0, 92.3)
- moved R6 25.4 mm to (130.0, 83.4)
- moved SW1 25.4 mm to (145.2, 127.0)
- moved SW2 25.4 mm to (135.5, 127.0)
- moved SW3 25.4 mm to (78.7, 127.0)
- moved SW4 25.4 mm to (88.9, 127.0)
- moved U1 25.4 mm to (114.3, 106.7)
- moved C1 25.4 mm to (104.1, 50.8)
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Routing:
- net /CONC-: track 0.00 -> 154.1 mm
- net /CONC+: track 0.00 -> 152.6 mm
- net /VCCD: track 0.00 -> 144.4 mm
- net /TXD: track 0.00 -> 139.7 mm
- net /GNDC: track 0.00 -> 139.1 mm
- net /COND-: track 0.00 -> 139.0 mm
- net /COND+: track 0.00 -> 136.9 mm
- net /RXD: track 0.00 -> 135.0 mm
- net /RXC: track 0.00 -> 134.4 mm
- net /GNDD: track 0.00 -> 130.4 mm
- net /TXC: track 0.00 -> 129.7 mm
- net /VCCC: track 0.00 -> 125.1 mm
- net /CONB-: track 0.00 -> 58.8 mm
- net /CONB+: track 0.00 -> 58.8 mm
- net /RXB: track 0.00 -> 54.1 mm
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Other:
- board size 88.9 x 88.9 mm -> 114.3 x 114.3 mm
- board text removed: "ASTAR TECH"
- board text removed: "by Greatreyhan"
