File: PCB_Sensor.kicad_sch (KiCad schematic)
At the start: 38 parts, among them J1 DHT22, J10 PRGM, J11 UWB, J12 LCDDATA, J13 LCDTOUCH, J14 ESP01A, J15 ESP01B, J2 VOLTSENSOR, J4 COM, J5 ALERT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

Commit message: update
Parts:
- added J16: DRV_B, TerminalBlock:TerminalBlock_bornier-2_P5.08mm, symbol Connector:Screw_Terminal_01x02
- added J17: DRV_C, TerminalBlock:TerminalBlock_bornier-2_P5.08mm, symbol Connector:Screw_Terminal_01x02
- added J18: DRV_D, TerminalBlock:TerminalBlock_bornier-2_P5.08mm, symbol Connector:Screw_Terminal_01x02
- added J19: MTR_A, TerminalBlock:TerminalBlock_bornier-2_P5.08mm, symbol Connector:Screw_Terminal_01x02
- added J20: MTR_B, TerminalBlock:TerminalBlock_bornier-2_P5.08mm, symbol Connector:Screw_Terminal_01x02
- added J21: MTR_C, TerminalBlock:TerminalBlock_bornier-2_P5.08mm, symbol Connector:Screw_Terminal_01x02
- added J22: MTR_D, TerminalBlock:TerminalBlock_bornier-2_P5.08mm, symbol Connector:Screw_Terminal_01x02
- added J23: DRV_ENCA, Connector_PinHeader_2.54mm:PinHeader_1x04_P2.54mm_Vertical, symbol Connector:Conn_01x04_Socket
- added J24: DRV_ENCB, Connector_PinHeader_2.54mm:PinHeader_1x04_P2.54mm_Vertical, symbol Connector:Conn_01x04_Socket
- added J25: DRV_ENCC, Connector_PinHeader_2.54mm:PinHeader_1x04_P2.54mm_Vertical, symbol Connector:Conn_01x04_Socket
- added J26: DRV_ENCD, Connector_PinHeader_2.54mm:PinHeader_1x04_P2.54mm_Vertical, symbol Connector:Conn_01x04_Socket
- added J27: ENCA, Connector_PinHeader_2.54mm:PinHeader_1x04_P2.54mm_Vertical, symbol Connector:Conn_01x04_Socket
- added J28: ENCC, Connector_PinHeader_2.54mm:PinHeader_1x04_P2.54mm_Vertical, symbol Connector:Conn_01x04_Socket
- added J29: ENCB, Connector_PinHeader_2.54mm:PinHeader_1x04_P2.54mm_Vertical, symbol Connector:Conn_01x04_Socket
- added J3: DRV_A, TerminalBlock:TerminalBlock_bornier-2_P5.08mm, symbol Connector:Screw_Terminal_01x02
- added J30: ENCD, Connector_PinHeader_2.54mm:PinHeader_1x04_P2.54mm_Vertical, symbol Connector:Conn_01x04_Socket
Connections:
- new net CONA+: J19.1 (Pin_1), J3.1 (Pin_1)
- new net CONA-: J19.2 (Pin_2), J3.2 (Pin_2)
- new net CONB+: J16.1 (Pin_1), J20.1 (Pin_1)
- new net CONB-: J16.2 (Pin_2), J20.2 (Pin_2)
- new net CONC+: J17.1 (Pin_1), J21.1 (Pin_1)
- new net CONC-: J17.2 (Pin_2), J21.2 (Pin_2)
- new net COND+: J18.1 (Pin_1), J22.1 (Pin_1)
- new net COND-: J18.2 (Pin_2), J22.2 (Pin_2)
- new net GNDA: J23.4 (Pin_4), J27.4 (Pin_4)
- new net GNDB: J24.4 (Pin_4), J29.4 (Pin_4)
- new net GNDC: J25.4 (Pin_4), J28.4 (Pin_4)
- new net GNDD: J26.4 (Pin_4), J30.4 (Pin_4)
- new net RXA: J23.3 (Pin_3), J27.3 (Pin_3)
- new net RXB: J24.3 (Pin_3), J29.3 (Pin_3)
- new net RXC: J25.3 (Pin_3), J28.3 (Pin_3)
- new net RXD: J26.3 (Pin_3), J30.3 (Pin_3)
- new net TXA: J23.2 (Pin_2), J27.2 (Pin_2)
- new net TXB: J24.2 (Pin_2), J29.2 (Pin_2)
- new net TXC: J25.2 (Pin_2), J28.2 (Pin_2)
- new net TXD: J26.2 (Pin_2), J30.2 (Pin_2)
- new net VCCA: J23.1 (Pin_1), J27.1 (Pin_1)
- new net VCCB: J24.1 (Pin_1), J29.1 (Pin_1)
- new net VCCC: J25.1 (Pin_1), J28.1 (Pin_1)
- new net VCCD: J26.1 (Pin_1), J30.1 (Pin_1)
Other:
- note added: "Driver_Connector"
- note added: "Driver_Encoder"
- note added: "Motor_Connector"
